Commit message: deleted kite planner scenes, obstacles movable, nicer objects, nicer robo config, collision between obstacles ignored

File: models/ball.urdf (robot description, URDF)
Before this commit: robot sphere, 1 links, 0 joints
Links:
- link sphere: geometry collision sphere radius=0.12; visual mesh filename=ball.glb

File: models/cocube.urdf (robot description, URDF)
Before this commit: robot box, 1 links, 0 joints
Links:
- link box: geometry collision box size=.7 .7 .7; visual mesh filename=cocube.glb

File: models/pallet.urdf (robot description, URDF)
Before this commit: robot box, 1 links, 0 joints
Links:
- link box: geometry collision box size=1.2 0.8 0.144; visual mesh filename=pallet.glb

File: models/rubik.urdf (robot description, URDF)
Before this commit: robot box, 1 links, 0 joints
Links:
- link box: geometry collision box size=.065 .065 .065; visual mesh filename=rubik.glb
